Commit message: robotic arm code added

File: src/my_robot_description/urdf/common_properties.xacro (robot description, xacro)
@@ -6,4 +6,10 @@
     <material name="gray">
         <color rgba="0.5 0.5 0.5 1" />
+    </material>
+    <material name="orange">
+        <color rgba="1.0 0.5 0 1" />
+    </material>
+    <material name="yellow" >
+        <color rgba="1.0 1.0 0 1" />
     </material>
     <xacro:macro name="box_inertia" params="m l w h xyz rpy">

File: src/my_robot_description/urdf/mobile_base_gazebo.xacro (robot description, xacro)
@@ -12,4 +12,6 @@
     <gazebo reference="caster_wheel_link">
         <material>Gazebo/Grey</material>
+        <mul value="0.1" />
+        <mu2 value="0.1" />
     </gazebo>
     <!-- we are added new plugin ros difference driver -->

File: src/my_robot_description/urdf/second_robot.urdf.xacro (robot description, xacro)
@@ -4,3 +4,12 @@
     <xacro:include filename="mobile_base.xacro" />
     <xacro:include filename="mobile_base_gazebo.xacro" />
+    <xacro:include filename="robotic_arm.xacro" />
+    <xacro:include filename="robotic_arm_gazebo.xacro" />
+    <joint name="mobile_base_arm_joint" type="fixed" >
+        <parent link="base_link" />
+        <child link="arm_base_link" />
+        <origin xyz="${base_length / 4.0} 0 ${base_height}" rpy="0 0 0" />
+    </joint>
+    <!-- Camera include -->
+    <!-- <xacro:include filename="camera.xacro" /> -->
 </robot>
